File: taro60.kicad_pcb (KiCad board)
At the start: 2 copper layers, 285.8 x 95.2 mm, 144 parts, among them SW1 SW_Push, U1 ATmega32U4-AU, Y1 16MHz

Commit message: pcb finished
Routing:
- added copper zone on B.Cu, net GND
Changed lines of the file:
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@@
   (segment (start 82.01875 113.825) (end 82.01875 114.929) (width 0.254) (layer F.Cu) (net 103))
   (segment (start 82.01875 121.125) (end 86.51875 121.125) (width 0.254) (layer F.Cu) (net 103))
+  (zone (net 1) (net_name GND) (layer B.Cu) (hatch edge 0.508)
+    (connect_pads (clearance 0.508))
+    (min_thickness 0.254)
+    (fill yes (arc_segments 32) (thermal_gap 0.508) (thermal_bridge_width 0.508))
+    (polygon
+      (pts
+        (xy 143.66875 150.8125) (xy 143.66875 173.83125) (xy 171.45 173.83125) (xy 171.45 150.8125)
+      )
+    )
+  )
+  (zone (net 1) (net_name GND) (layer B.Cu) (hatch edge 0.508)
+    (connect_pads (clearance 0.508))
+    (min_thickness 0.254)
+    (fill yes (arc_segments 32) (thermal_gap 0.508) (thermal_bridge_width 0.508))
+    (polygon
+      (pts
+        (xy 78.58125 112.7125) (xy 78.58125 122.2375) (xy 91.28125 122.2375) (xy 91.28125 112.7125)
+      )
+    )
+  )
 )
