File: taro60.kicad_pcb (KiCad board)
At the start: 2 copper layers, 285.8 x 95.2 mm, 144 parts, among them SW1 SW_Push, U1 ATmega32U4-AU, Y1 16MHz

Commit message: updated pcb
Parts:
- removed USB1: Molex-0548190589, random-keyboard-parts:Molex-0548190589
- added J1: Conn_01x04_Female, Connector_Molex:Molex_CLIK-Mate_502382-0470_1x04-1MP_P1.25mm_Vertical, B.Cu at (84.9, 117.5)
Connections:
- F1 pad 2: VCC -> VBUS
Routing:
- net VCC: track 31.6 -> 0.00 mm, vias 2 -> 0
- net VBUS: track 0.00 -> 28.4 mm, vias 0 -> 2
- net Net-(USB1-Pad6): track 16.3 -> 0.00 mm
- net GND: track 396.8 -> 399.2 mm
- net D+: track 83.2 -> 84.9 mm
- net D-: track 84.3 -> 82.9 mm
